File: pcb/reversible_split.kicad_pcb (KiCad board)
At the start: 2 copper layers, 134 x 93.8 mm, 22 parts

Commit message: Manually flipped mc footprint
The ergogen footprint for the mcu seems buggy.
Parts:
- JST1, MCU1: moved to B.Cu
Connections:
- JST1 pad 2: B- -> GND
Routing:
- net pos: track 0.00 -> 19.2 mm, vias 0 -> 2
- net GND: track 29.5 -> 40.0 mm, vias 0 -> 1
- net RST: track 9.84 -> 20.3 mm, vias 0 -> 1

Commit message: Routed quick and dirty
Parts:
- moved RST1 4.42 mm to (165.5, 127.8)
- moved S7 4.42 mm to (158.5, 58.1)
- moved S1 4.42 mm to (122.5, 103.6)
- moved S17 4.42 mm to (209.3, 119.1)
- moved S5 4.42 mm to (161.8, 96.1)
- moved S12 4.42 mm to (200.8, 78.1)
- moved S3 4.42 mm to (139.9, 94.1)
- moved MCU1 4.42 mm to (181.8, 113.1)
- moved S11 4.42 mm to (200.8, 97.2)
- moved S13 4.42 mm to (200.8, 59.1)
- moved S18 4.42 mm to (231.5, 122.0)
- moved PWR1 4.42 mm to (196.1, 128.0)
- moved S2 4.42 mm to (143.9, 112.7)
- moved S15 4.42 mm to (219.8, 80.0)
- moved S8 4.42 mm to (181.8, 89.6)
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Routing:
- net GND: track 40.0 -> 839.1 mm, vias 1 -> 7
- net matrix_ring_top: track 9.84 -> 171.0 mm, vias 0 -> 3
- net matrix_inner_top: track 9.84 -> 146.3 mm, vias 0 -> 6
- net matrix_inner_home: track 9.84 -> 131.7 mm, vias 0 -> 6
- net matrix_middle_top: track 9.84 -> 126.8 mm, vias 0 -> 1
- net matrix_outer_home: track 9.83 -> 123.0 mm, vias 0 -> 1
- net thumb_tucky: track 9.83 -> 120.2 mm, vias 0 -> 6
- net thumb_reachy: track 9.83 -> 117.3 mm, vias 0 -> 5
- net matrix_pinky_top: track 9.83 -> 114.5 mm, vias 0 -> 2
- net matrix_ring_home: track 9.83 -> 109.1 mm, vias 0 -> 1
- net matrix_middle_home: track 9.84 -> 102.0 mm, vias 0 -> 2
- net matrix_index_top: track 9.84 -> 98.0 mm, vias 0 -> 1
- net matrix_middle_bottom: track 9.84 -> 92.8 mm, vias 0 -> 1
- net matrix_pinky_home: track 9.83 -> 90.3 mm, vias 0 -> 3
- net matrix_ring_bottom: track 9.83 -> 88.3 mm, vias 0 -> 1
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Other:
- outline, holes or cut-outs redrawn

Commit message: Final production files
Routing:
- net matrix_inner_bottom: vias 5 -> 4
Other:
- board text added: "by jfelixh"

Commit message: Reverted name change
Other:
- board text added: "SplayBreak v2.0.0"
- board text removed: "WingSpan v2.0.0"
Changed lines of the file:
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@@
 		(fp_arc
 			(start -2.484999 -0.920001)
-			(mid -1.74436 -2.328061)
+			(mid -1.74436 -2.328062)
 			(end -0.225 -2.8)
 			(stroke
@@
 		(fp_arc
 			(start -2.484999 -0.920001)
-			(mid -1.74436 -2.328061)
+			(mid -1.74436 -2.328062)
 			(end -0.225 -2.8)
 			(stroke
@@
 		(fp_arc
 			(start 2.28 7.449999)
-			(mid 2.595906 6.487327)
+			(mid 2.595905 6.487326)
 			(end 3.5 6.03)
 			(stroke
@@
 		(fp_arc
 			(start -2.484999 -0.920001)
-			(mid -1.74436 -2.328061)
+			(mid -1.74436 -2.328062)
 			(end -0.225 -2.8)
 			(stroke
@@
 		(layer "Edge.Cuts")
 	)
-	(gr_text "WingSpan v2.0.0"
+	(gr_text "SplayBreak v2.0.0"
 		(at 158.914987 123.845521 0)
 		(layer "B.SilkS")
@@
 	)
 	(gr_text "by jfelixh"
-		(at 157.4 127.8 0)
+		(at 159.2 127.8 0)
 		(layer "B.SilkS")
 		(effects
@@
 	)
 	(gr_text "by jfelixh"
-		(at 146.4 127.8 0)
+		(at 148.2 127.8 0)
 		(layer "F.SilkS")
 		(effects
@@
 		)
 	)
-	(gr_text "WingSpan v2.0.0"
+	(gr_text "SplayBreak v2.0.0"
 		(at 158.914987 123.845521 0)
 		(layer "F.SilkS")

Commit message: Regenerated build files with updated text
Other:
- board text added: "by flhps"
- board text removed: "by jfelixh"
